Commit message: Added camera and end plates to trough.

File: urdf/trough.urdf.xacro (robot description, xacro)
@@ -13,4 +13,12 @@
     <xacro:property name="trough_long_width" value="0.1"/>
     <xacro:property name="trough_long_height" value="0.01"/>
+    <xacro:property name="trough_short_mass" value="0.010"/>
+    <xacro:property name="trough_short_length" value="0.1"/>
+    <xacro:property name="trough_short_width" value="0.1"/>
+    <xacro:property name="trough_short_height" value="0.01"/>
+    <xacro:property name="camera_mass" value="0.500"/>
+    <xacro:property name="camera_length" value="0.10"/>
+    <xacro:property name="camera_width" value="0.10"/>
+    <xacro:property name="camera_height" value="0.10"/>
     <xacro:include filename="$(find rl_wheel)/urdf/macros.xacro"/>
     <xacro:include filename="$(find rl_wheel)/urdf/materials.xacro"/>
@@ -93,4 +101,50 @@
         </visual>
     </link>
+    <link name="trough_left">
+        <xacro:box_inertial name="trough_left"
+            m="${trough_short_mass}"
+            x="${trough_short_length}" y="${trough_short_width}" z="${trough_short_height}"/>
+        <collision name='trough_left_collision'>
+            <geometry>
+                <box size="${trough_short_length} ${trough_short_width} ${trough_short_height}"/>
+            </geometry>
+        </collision>
+        <visual name='trough_left_visual'>
+            <origin xyz="0 0 0" rpy=" 0 0 0"/>
+            <geometry>
+                <box size="${trough_short_length} ${trough_short_width} ${trough_short_height}"/>
+            </geometry>
+        </visual>
+    </link>
+        <link name="trough_right">
+        <xacro:box_inertial name="trough_left"
+            m="${trough_short_mass}"
+            x="${trough_short_length}" y="${trough_short_width}" z="${trough_short_height}"/>
+        <collision name='trough_left_collision'>
+            <geometry>
+                <box size="${trough_short_length} ${trough_short_width} ${trough_short_height}"/>
+            </geometry>
+        </collision>
+        <visual name='trough_left_visual'>
+            <origin xyz="0 0 0" rpy=" 0 0 0"/>
+            <geometry>
+                <box size="${trough_short_length} ${trough_short_width} ${trough_short_height}"/>
+            </geometry>
+        </visual>
+    </link>
+    <link name="camera_link">
+        <xacro:box_inertial name="camera"
+            m="${camera_mass}" x="${camera_length}" y="${camera_width}" z="${camera_height}"/>
+        <visual>
+            <geometry>
+                <box size="${camera_width} ${camera_height} ${camera_length}"/>
+            </geometry>
+        </visual>
+        <collision>
+            <geometry>
+                <box size="${camera_width} ${camera_height} ${camera_length}"/>
+            </geometry>
+        </collision>
+    </link>
     <!-- *** JOINTS *** -->
     <joint name="base_arm_joint" type="fixed">
@@ -118,9 +172,70 @@
         <origin xyz="0 0 ${trough_long_width}"/>
     </joint>
+    <joint name="trough_back_left_joint" type="fixed">
+        <parent link="trough_back"/>
+        <child link="trough_left"/>
+        <origin xyz="${trough_long_length/2} 0 ${trough_long_width/2}"
+                rpy="0 1.57 0"/>
+    </joint>
+    <joint name="trough_back_right_joint" type="fixed">
+        <parent link="trough_back"/>
+        <child link="trough_right"/>
+        <origin xyz="${-trough_long_length/2} 0 ${trough_long_width/2}"
+                rpy="0 1.57 0"/>
+    </joint>
+    <joint name="camera_base_joint" type="fixed">
+        <parent link="base_link"/>
+        <child link="camera_link"/>
+        <origin xyz="0.1 0 1" rpy="0 1.57 0"/>
+    </joint>
+    <!-- *** MATERIAL *** -->
     <gazebo reference="base_link">
-        <material>grey</material>
+        <material>Gazebo/Green</material>
     </gazebo>
     <gazebo reference="arm_link">
-        <material>Gazebo/Orange</material>
+        <material>Gazebo/Red</material>
     </gazebo>
+    <gazebo reference="ball_link">
+        <material>Gazebo/Blue</material>
+    </gazebo>
+    <!-- CAMERA PLUGIN -->
+    <gazebo reference="camera_link">
+        <sensor type="camera" name="camera1">
+        <update_rate>30.0</update_rate>
+        <camera name="head">
+            <horizontal_fov>1.3962634</horizontal_fov>
+            <image>
+            <width>800</width>
+            <height>800</height>
+            <format>R8G8B8</format>
+            </image>
+            <clip>
+            <near>0.02</near>
+            <far>300</far>
+            </clip>
+            <noise>
+            <type>gaussian</type>
+            <!-- Noise is sampled independently per pixel on each frame.
+                That pixel's noise value is added to each of its color
+                channels, which at that point lie in the range [0,1]. -->
+            <mean>0.0</mean>
+            <stddev>0.007</stddev>
+            </noise>
+        </camera>
+        <plugin name="camera_controller" filename="libgazebo_ros_camera.so">
+            <alwaysOn>true</alwaysOn>
+            <updateRate>0.0</updateRate>
+            <cameraName>rrbot/camera1</cameraName>
+            <imageTopicName>image_raw</imageTopicName>
+            <cameraInfoTopicName>camera_info</cameraInfoTopicName>
+            <frameName>camera_link</frameName>
+            <hackBaseline>0.07</hackBaseline>
+            <distortionK1>0.0</distortionK1>
+            <distortionK2>0.0</distortionK2>
+            <distortionK3>0.0</distortionK3>
+            <distortionT1>0.0</distortionT1>
+            <distortionT2>0.0</distortionT2>
+        </plugin>
+        </sensor>
+  </gazebo>
 </robot>

Commit message: Added joint controller for trough.

File: urdf/trough.urdf.xacro (robot description, xacro)
@@ -23,5 +23,7 @@
     <xacro:include filename="$(find rl_wheel)/urdf/macros.xacro"/>
     <xacro:include filename="$(find rl_wheel)/urdf/materials.xacro"/>
-    <link name="base_link">
+    <!-- Use the world link to fix the platform_base_link to the Gazebo base_link-->
+    <link name="world"/>
+    <link name="platform_base_link">
         <xacro:box_inertial name="base"
             m="${base_mass}" x="${base_length}" y="${base_width}" z="${base_height}"/>
@@ -148,6 +150,10 @@
     </link>
     <!-- *** JOINTS *** -->
+    <joint name="fixed" type="fixed">
+        <parent link="world"/>
+        <child link="platform_base_link"/>
+    </joint>
     <joint name="base_arm_joint" type="fixed">
-        <parent link="base_link"/>
+        <parent link="platform_base_link"/>
         <child link="arm_link"/>
         <origin xyz="0.2 0 ${arm_height/2}"
@@ -185,17 +191,14 @@
     </joint>
     <joint name="camera_base_joint" type="fixed">
-        <parent link="base_link"/>
+        <parent link="platform_base_link"/>
         <child link="camera_link"/>
         <origin xyz="0.1 0 1" rpy="0 1.57 0"/>
     </joint>
     <!-- *** MATERIAL *** -->
-    <gazebo reference="base_link">
-        <material>Gazebo/Green</material>
+    <gazebo reference="platform_base_link">
+        <material>Gazebo/Blue</material>
     </gazebo>
     <gazebo reference="arm_link">
         <material>Gazebo/Red</material>
-    </gazebo>
-    <gazebo reference="ball_link">
-        <material>Gazebo/Blue</material>
     </gazebo>
     <!-- CAMERA PLUGIN -->
@@ -206,19 +209,19 @@
             <horizontal_fov>1.3962634</horizontal_fov>
             <image>
-            <width>800</width>
-            <height>800</height>
-            <format>R8G8B8</format>
+                <width>800</width>
+                <height>800</height>
+                <format>R8G8B8</format>
             </image>
             <clip>
-            <near>0.02</near>
-            <far>300</far>
+                <near>0.02</near>
+                <far>300</far>
             </clip>
             <noise>
-            <type>gaussian</type>
-            <!-- Noise is sampled independently per pixel on each frame.
-                That pixel's noise value is added to each of its color
-                channels, which at that point lie in the range [0,1]. -->
-            <mean>0.0</mean>
-            <stddev>0.007</stddev>
+                <type>gaussian</type>
+                <!-- Noise is sampled independently per pixel on each frame.
+                    That pixel's noise value is added to each of its color
+                    channels, which at that point lie in the range [0,1]. -->
+                <mean>0.0</mean>
+                <stddev>0.007</stddev>
             </noise>
         </camera>
@@ -226,5 +229,5 @@
             <alwaysOn>true</alwaysOn>
             <updateRate>0.0</updateRate>
-            <cameraName>rrbot/camera1</cameraName>
+            <cameraName>camera1</cameraName>
             <imageTopicName>image_raw</imageTopicName>
             <cameraInfoTopicName>camera_info</cameraInfoTopicName>
@@ -238,4 +241,25 @@
         </plugin>
         </sensor>
-  </gazebo>
+    </gazebo>
+    <!-- TRANSMISSIONS -->
+    <transmission name="trough_tran">
+        <type>transmission_interface/SimpleTransmission</type>
+        <joint name="arm_trough_back_joint">
+            <hardwareInterface>
+                hardware_interface/EffortJointInterface
+            </hardwareInterface>
+        </joint>
+        <actuator name="motor1">
+            <hardwareInterface>
+                hardware_interface/EffortJointInterface
+            </hardwareInterface>
+            <mechanicalReduction>1</mechanicalReduction>
+        </actuator>
+    </transmission>
+    <gazebo>
+        <plugin name="gazebo_ros_control" filename="libgazebo_ros_control.so">
+            <robotNamespace>/trough_bot</robotNamespace>
+            <robotSimType>gazebo_ros_control/DefaultRobotHWSim</robotSimType>
+        </plugin>
+    </gazebo>
 </robot>

Commit message: We can control trough using rqt_gui interface

File: urdf/trough.urdf.xacro (robot description, xacro)
@@ -166,4 +166,5 @@
             rpy="-1.57 0 1.57"/>
         <axis xyz="0 0 -1"/>
+        <dynamics damping="0.0" friction="0.2"/>
     </joint>
     <joint name="trough_back_floor_joint" type="fixed">
