Commit message: First implementation of ball controller. Control loop time has high jitter.

File: urdf/ball.urdf.xacro (robot description, xacro)
@@ -1,5 +1,5 @@
 <?xml version="1.0"?>
 <robot name="ball" xmlns:xacro="http://www.ros.org/wiki/xacro">
-    <xacro:property name="ball_mass" value="0.500"/>
+    <xacro:property name="ball_mass" value="0.50"/>
     <xacro:property name="ball_radius" value="0.02"/>
     <xacro:include filename="$(find rl_wheel)/urdf/macros.xacro"/>

File: urdf/trough.urdf.xacro (robot description, xacro)
@@ -10,5 +10,5 @@
     <xacro:property name="arm_height" value="0.5"/>
     <xacro:property name="trough_long_mass" value="0.100"/>
-    <xacro:property name="trough_long_length" value="0.3"/>
+    <xacro:property name="trough_long_length" value="0.5"/>
     <xacro:property name="trough_long_width" value="0.1"/>
     <xacro:property name="trough_long_height" value="0.01"/>
@@ -64,5 +64,5 @@
             </geometry>
         </collision>
-        <visual name='trough_long_visual'>
+        <visual name='trough_back_visual'>
             <origin xyz="0 0 0" rpy=" 0 0 0"/>
             <geometry>
@@ -72,13 +72,21 @@
     </link>
     <link name="trough_floor">
-        <xacro:box_inertial name="trough_back"
+        <xacro:box_inertial name="trough_floor"
             m="${trough_long_mass}"
             x="${trough_long_length}" y="${trough_long_width}" z="${trough_long_height}"/>
-        <collision name='trough_back_collision'>
-            <geometry>
-                <box size="${trough_long_length} ${trough_long_width} ${trough_long_height}"/>
-            </geometry>
-        </collision>
-        <visual name='trough_long_visual'>
+        <collision name='trough_floor_collision'>
+            <geometry>
+                <box size="${trough_long_length} ${trough_long_width} ${trough_long_height}"/>
+            </geometry>
+            <!-- <surface>
+                <friction>
+                    <ode>
+                        <mu>10</mu>
+                        <mu2>10</mu2>
+                    </ode>
+                </friction>
+            </surface> -->
+        </collision>
+        <visual name='trough_floor_visual'>
             <origin xyz="0 0 0" rpy=" 0 0 0"/>
             <geometry>
@@ -120,13 +128,13 @@
     </link>
         <link name="trough_right">
-        <xacro:box_inertial name="trough_left"
+        <xacro:box_inertial name="trough_right"
             m="${trough_short_mass}"
             x="${trough_short_length}" y="${trough_short_width}" z="${trough_short_height}"/>
-        <collision name='trough_left_collision'>
-            <geometry>
-                <box size="${trough_short_length} ${trough_short_width} ${trough_short_height}"/>
-            </geometry>
-        </collision>
-        <visual name='trough_left_visual'>
+        <collision name='trough_right_collision'>
+            <geometry>
+                <box size="${trough_short_length} ${trough_short_width} ${trough_short_height}"/>
+            </geometry>
+        </collision>
+        <visual name='trough_right_visual'>
             <origin xyz="0 0 0" rpy=" 0 0 0"/>
             <geometry>
@@ -138,10 +146,10 @@
         <xacro:box_inertial name="camera"
             m="${camera_mass}" x="${camera_length}" y="${camera_width}" z="${camera_height}"/>
-        <visual>
+        <visual name="camera_visual">
             <geometry>
                 <box size="${camera_width} ${camera_height} ${camera_length}"/>
             </geometry>
         </visual>
-        <collision>
+        <collision name="camera_collision">
             <geometry>
                 <box size="${camera_width} ${camera_height} ${camera_length}"/>
@@ -194,11 +202,16 @@
         <parent link="platform_base_link"/>
         <child link="camera_link"/>
-        <origin xyz="0.1 0 1" rpy="0 1.57 0"/>
+        <origin xyz="0.1 0 0.8" rpy="0 1.57 0"/>
     </joint>
     <!-- *** MATERIAL *** -->
     <gazebo reference="platform_base_link">
-        <material>Gazebo/Blue</material>
+        <material>Gazebo/Green</material>
     </gazebo>
     <gazebo reference="arm_link">
+        <material>Gazebo/Red</material>
+    </gazebo>
+    <gazebo reference="trough_floor">
+        <mu1>10</mu1>
+        <mu2>10</mu2>
         <material>Gazebo/Red</material>
     </gazebo>
@@ -206,10 +219,10 @@
     <gazebo reference="camera_link">
         <sensor type="camera" name="camera1">
-        <update_rate>30.0</update_rate>
+        <update_rate>10.0</update_rate>
         <camera name="head">
             <horizontal_fov>1.3962634</horizontal_fov>
             <image>
                 <width>800</width>
-                <height>800</height>
+                <height>400</height>
                 <format>R8G8B8</format>
             </image>

Commit message: Implemented a ball position PID controller (somewhat underdamped)

File: urdf/ball.urdf.xacro (robot description, xacro)
@@ -1,5 +1,5 @@
 <?xml version="1.0"?>
 <robot name="ball" xmlns:xacro="http://www.ros.org/wiki/xacro">
-    <xacro:property name="ball_mass" value="0.50"/>
+    <xacro:property name="ball_mass" value="0.10"/>
     <xacro:property name="ball_radius" value="0.02"/>
     <xacro:include filename="$(find rl_wheel)/urdf/macros.xacro"/>

File: urdf/trough.urdf.xacro (robot description, xacro)
@@ -219,5 +219,5 @@
     <gazebo reference="camera_link">
         <sensor type="camera" name="camera1">
-        <update_rate>10.0</update_rate>
+        <update_rate>30.0</update_rate>
         <camera name="head">
             <horizontal_fov>1.3962634</horizontal_fov>
